File: single-drive_pcb/single-drive_pcb.kicad_pcb (KiCad board)
At the start: 2 copper layers, 0 parts

Commit message: started on pcb layout, need some dimensions before continuing
Parts:
- added BT1: LIPO, JST_PH_2-pin, F.Cu at (132.1, 101.6)
- added C1: 22pF, 0603(1608m), F.Cu at (139.3, 82.8)
- added C10: 1uF, 0603(1608m), F.Cu at (145.2, 84.3)
- added C11: 2.2uF, 0603(1608m), F.Cu at (136.4, 84.3)
- added C12: 470pF, 0603(1608m), F.Cu at (139.3, 84.3)
- added C13: 10uF, 0603(1608m), F.Cu at (165.7, 82.8)
- added C14: 1uF, 0603(1608m), F.Cu at (162.8, 82.8)
- added C2: 22pF, 0603(1608m), F.Cu at (145.2, 82.8)
- added C3: 1uF, 0603(1608m), F.Cu at (151.0, 82.8)
- added C4: 0.01uF, 0603(1608m), F.Cu at (124.7, 84.3)
- added C5: 2.2uF, 0603(1608m), F.Cu at (171.6, 82.8)
- added C6: 10uF, 0603(1608m), F.Cu at (130.6, 84.3)
- added C7: 1uF, 0603(1608m), F.Cu at (153.9, 82.8)
- added C8: 1uF, 0603(1608m), F.Cu at (136.4, 82.8)
- added C9: 1uF, 0603(1608m), F.Cu at (159.9, 82.8)
- added F1: 500mA, 1206(3216m), F.Cu at (139.7, 95.9)
- added IC1: MCP4232, MSOP10, F.Cu at (147.3, 121.3)
- added IC2: ATMEGA328P_TQFP, TQFP32_7mm, F.Cu at (149.9, 96.5)
- added IC3: DRV8834_SOP, HTSSOP24, F.Cu at (149.9, 114.3)
- added IC4: MIC5205, SOT23-5, F.Cu at (139.7, 103.5)
- added IC5: BLE112-A, BLE112-A, F.Cu at (165.1, 106.7)
- added IC6: MAX1555, SOT23-5, F.Cu at (139.7, 99.7)
- added J1: MICROUSB, MICROUSB_sm, F.Cu at (121.9, 111.8)
- added LED1: L1, 0603(1608m)_led, F.Cu at (161.0, 79.5)
- added LED2: L2, 0603(1608m)_led, F.Cu at (158.1, 79.5)
- added LED3: PWR, 0603(1608m)_led, F.Cu at (166.9, 79.5)
- added LED4: CHG, 0603(1608m)_led, F.Cu at (164.0, 79.5)
- added M1: STEPPER, SIP4, F.Cu at (164.5, 121.3)
- added P1: AVR_ISP, 2x3-array, F.Cu at (130.2, 121.3)
- added P2: CC_ISP, 2x5-array, F.Cu at (177.8, 116.8)
- added R1: 10kΩ, 0603(1608m), F.Cu at (142.2, 82.8)
- added R10: 10kΩ, 0603(1608m), F.Cu at (172.7, 79.0)
- added R11: 1kΩ, 0603(1608m), F.Cu at (127.6, 84.3)
- added R12: 1kΩ, 0603(1608m), F.Cu at (168.7, 82.8)
- added R13: 10kΩ, 0603(1608m), F.Cu at (142.2, 84.3)
- added R2: 10kΩ, 0603(1608m), F.Cu at (148.1, 82.8)
- added R3: 1kΩ, 0603(1608m), F.Cu at (133.5, 82.8)
- added R4: 1kΩ, 0603(1608m), F.Cu at (127.6, 82.8)
- added R5: 10kΩ, 0603(1608m), F.Cu at (133.5, 84.3)
- added R6: 10kΩ, 0603(1608m), F.Cu at (124.7, 82.8)
- added R7: 22kΩ, 0603(1608m), F.Cu at (157.0, 82.8)
- added R8: 10kΩ, 0603(1608m), F.Cu at (169.8, 79.0)
- added R9: 10kΩ, 0603(1608m), F.Cu at (130.6, 82.8)
- added S1: RST, SPST_4-pin-sm, F.Cu at (130.2, 111.8)
- added S2: BT_RST, SPST_4-pin-sm, F.Cu at (177.8, 106.0)
- added VR1: 10Ω, BOURNS-3362P_pot, F.Cu at (138.4, 111.1)
- added VR2: 10Ω, BOURNS-3362P_pot, F.Cu at (138.4, 119.4)
- added Y1: 8MHz, HC49, F.Cu at (149.9, 106.7)

Commit message: trying out some stuff
Parts:
- added M2: VAL**, M2, F.Cu at (110.4, 142.2)
- added M2: VAL**, M2, F.Cu at (85.2, 137.0)
- moved M1 102.9 mm to (63.5, 141.0)
- moved C14 100.6 mm to (67.3, 114.3)
- moved LED1 90.8 mm to (83.6, 126.9), turned to 270 degrees
- moved LED2 86.7 mm to (85.5, 126.9), turned to 270 degrees
- moved IC3 84.9 mm to (67.1, 133.2), turned to 0 degrees
- moved C9 84.6 mm to (85.7, 123.4), turned to 270 degrees
- moved R10 84.3 mm to (104.4, 128.4), turned to 180 degrees
- moved IC2 81.0 mm to (77.3, 132.7), turned to 270 degrees
- moved R8 80.9 mm to (104.0, 126.1), turned to 135 degrees
- moved C7 79.1 mm to (98.7, 139.4), turned to 180 degrees
- moved C2 79.0 mm to (79.1, 126.1)
- moved S2 77.3 mm to (106.7, 136.3), turned to 45 degrees
- moved C1 76.8 mm to (75.9, 126.1)
- moved IC5 73.4 mm to (94.7, 127.6)
- moved Y1 72.8 mm to (78.7, 122.4), turned to 180 degrees
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Routing:
- net N-0000046: track 0.00 -> 59.3 mm
- net GND: track 0.00 -> 24.4 mm
- net VCC: track 0.00 -> 17.2 mm
- net N-0000055: track 0.00 -> 12.7 mm
- net N-0000054: track 0.00 -> 9.11 mm
- net N-0000043: track 0.00 -> 5.56 mm
- net N-0000031: track 0.00 -> 4.50 mm
- net N-0000042: track 0.00 -> 4.03 mm
- net N-0000036: track 0.00 -> 4.00 mm
- net /BT_RESET: track 0.00 -> 3.13 mm
- net N-0000045: track 0.00 -> 2.62 mm
- net N-0000044: track 0.00 -> 2.52 mm
Other:
- board outline added: 36.1 x 36.1 mm
- net class Default: via_dia 0.889 -> 0.762; via_drill 0.635 -> 0.381
- rule pad_to_mask_clearance: 0 -> 0.1778
- rule trace_min: 0.254 -> 0.1524
- rule via_min_drill: 0.508 -> 0.3302
- rule via_min_size: 0.889 -> 0.6858

Commit message: done for the day
Parts:
- added M3: VAL**, M3, F.Cu at (67.9, 152.4)
- added M3: VAL**, M3, F.Cu at (109.9, 152.4)
- IC5: moved to B.Cu
- moved M2 110.8 mm to (219.4, 122.2)
- moved R10 110.8 mm to (213.4, 108.4)
- moved R13 110.8 mm to (213.4, 110.0)
- moved R8 110.8 mm to (213.0, 106.1)
- moved R9 110.8 mm to (213.4, 111.8)
- moved S2 110.8 mm to (215.7, 116.3)
- moved C2 105.8 mm to (182.1, 102.1)
- moved M2 105.8 mm to (188.2, 113.0)
- moved R3 105.8 mm to (187.1, 106.7)
- moved Y1 105.8 mm to (181.7, 98.4)
- moved C1 105.8 mm to (178.9, 102.1)
- moved C7 105.8 mm to (201.7, 115.4)
- moved C8 105.8 mm to (188.7, 96.1)
- moved C9 105.8 mm to (188.7, 99.4)
- moved LED1 105.8 mm to (186.6, 102.9)
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Routing:
- net N-0000046: track 59.3 -> 0.00 mm
- net GND: track 24.4 -> 0.00 mm
- net VCC: track 17.2 -> 0.00 mm
- net N-0000055: track 12.7 -> 0.00 mm
- net N-0000054: track 9.11 -> 0.00 mm
- net N-0000043: track 5.56 -> 0.00 mm
- net N-0000031: track 4.50 -> 0.00 mm
- net N-0000042: track 4.03 -> 0.00 mm
- net N-0000036: track 4.00 -> 0.00 mm
- net /BT_RESET: track 3.13 -> 0.00 mm
- net N-0000045: track 2.62 -> 0.00 mm
- net N-0000044: track 2.52 -> 0.00 mm
Other:
- board outline removed

Commit message: board might actually work. or, you know, it might not
Parts:
- added M2: VAL**, M2, F.Cu at (88.9, 172.7)
- BT1: footprint JST_PH_2-pin -> JST_PH_2-pin_vert-sm
- C7, C8, C9, R10, R13, R9: moved to B.Cu
- Y1: footprint HC49 -> XTAL_TXC_7A
- moved M2 148.8 mm to (70.6, 123.8)
- moved S2 127.1 mm to (88.9, 125.3), turned to 180 degrees
- moved C2 121.6 mm to (67.3, 142.2), turned to 45 degrees
- moved R8 118.9 mm to (96.1, 128.0), turned to 0 degrees
- moved Y1 118.8 mm to (70.2, 139.3), turned to 315 degrees
- moved C1 117.9 mm to (68.6, 143.5), turned to 225 degrees
- moved R4 112.2 mm to (78.2, 126.1), turned to 270 degrees
- moved LED2 109.4 mm to (82.7, 130.6), turned to 180 degrees
- moved R3 108.8 mm to (80.0, 126.1), turned to 270 degrees
- moved LED1 107.0 mm to (82.7, 128.7), turned to 180 degrees
- moved LED4 102.7 mm to (81.8, 122.9), turned to 90 degrees
- moved C13 94.0 mm to (75.4, 119.5), turned to 90 degrees
- moved LED3 93.6 mm to (83.4, 122.9), turned to 270 degrees
- moved R13 92.9 mm to (120.8, 117.1)
- moved R9 92.9 mm to (120.8, 118.9)
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Routing:
- net GND: track 0.00 -> 114.6 mm
- net VCC: track 0.00 -> 70.9 mm
- net /RESET: track 0.00 -> 60.0 mm, vias 0 -> 2
- net N-0000011: track 0.00 -> 59.3 mm, vias 0 -> 2
- net /VBAT: track 0.00 -> 40.0 mm, vias 0 -> 2
- net /SCK: track 0.00 -> 29.3 mm, vias 0 -> 1
- net /MOSI: track 0.00 -> 25.6 mm, vias 0 -> 1
- net N-0000040: track 0.00 -> 25.1 mm
- net /MISO: track 0.00 -> 24.6 mm, vias 0 -> 1
- net N-0000020: track 0.00 -> 19.7 mm
- net N-0000039: track 0.00 -> 16.2 mm
- net N-0000042: track 0.00 -> 12.4 mm
- net N-0000016: track 0.00 -> 11.4 mm
- net /BT_RESET: track 0.00 -> 11.2 mm, vias 0 -> 1
- net N-0000055: track 0.00 -> 9.76 mm
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Other:
- net class Default: clearance 0.254 -> 0.1778; trace_width 0.254 -> 0.1778; via_dia 0.762 -> 0.6858; via_drill 0.381 -> 0.3302
- net class Motor added: clearance 0.254, trace_width 0.254, via_dia 0.762, via_drill 0.381
- rule trace_clearance: 0.254 -> 0.1778

Commit message: gonna take a break for a little while
Parts:
- turned M1 to 45 degrees
Routing:
- net N-0000028: track 0.00 -> 52.4 mm, vias 0 -> 1
- net N-0000032: track 0.00 -> 50.8 mm, vias 0 -> 1
- net N-0000029: track 0.00 -> 50.6 mm, vias 0 -> 1
- net /BT_RESET: track 11.2 -> 60.2 mm
- net N-0000015: track 0.00 -> 46.8 mm, vias 0 -> 1
- net N-0000046: track 0.00 -> 42.4 mm
- net /R_SEL: track 0.00 -> 36.4 mm
- net VCC: track 70.9 -> 82.4 mm, vias 0 -> 1
- net N-0000011: track 59.3 -> 63.4 mm
- net /DIR: track 0.00 -> 2.87 mm, vias 0 -> 1
- net /ENABLE: track 0.00 -> 2.27 mm, vias 0 -> 1
- net /STEP: track 0.00 -> 1.70 mm, vias 0 -> 1
- net N-0000040: track 25.1 -> 26.4 mm

Commit message: it's too late to be working on this
Parts:
- moved C9 85.6 mm to (77.0, 120.7), turned to 270 degrees
- moved C7 78.7 mm to (100.8, 133.2)
- moved C8 73.1 mm to (100.8, 131.6)
- moved R10 22.3 mm to (100.8, 125.3)
- moved R13 22.3 mm to (100.8, 127.0)
- moved R9 22.2 mm to (100.8, 128.7)
Connections:
- IC5 pad 13: N-0000046 (its old number) -> /AVR_RX
- IC5 pad 14: N-0000046 (its old number) -> /AVR_TX
- IC5 pad 15: N-0000046 (its old number) -> N-0000037
- IC5 pad 16: N-0000046 (its old number) -> N-0000037
- IC5 pad 17: N-0000046 (its old number) -> N-0000037
- IC5 pad 18: N-0000046 (its old number) -> N-0000037
- IC5 pad 19: N-0000046 (its old number) -> N-0000037
- IC5 pad 22: N-0000046 (its old number) -> N-0000037
- IC5 pad 23: N-0000046 (its old number) -> N-0000037
- IC5 pad 24: N-0000046 (its old number) -> N-0000037
- IC5 pad 25: /AVR_RX -> N-0000037
- IC5 pad 26: /AVR_TX -> N-0000037
- IC5 pad 6: N-0000046 (its old number) -> N-0000037
- IC5 pad 7: N-0000046 (its old number) -> N-0000037
- IC5 pad 8: N-0000046 (its old number) -> N-0000037
- R9 pad 1: N-0000046 (its old number) -> N-0000037
Routing:
- net N-000009: track 63.4 -> 2.56 mm, vias 2 -> 0
- net N-0000037: track 0.00 -> 52.0 mm
- net N-0000046 (its old number): track 42.4 -> 0.00 mm
- net /BT_DD: track 0.00 -> 36.0 mm
- net /BT_DC: track 0.00 -> 35.0 mm
- net GND: track 114.2 -> 144.9 mm
- net /ENABLE: track 2.27 -> 28.9 mm, vias 1 -> 2
- net VCC: track 82.4 -> 106.3 mm, vias 1 -> 0
- net /AVR_RX: track 0.00 -> 18.1 mm, vias 0 -> 1
- net N-0000032: track 0.00 -> 18.0 mm
- net /AVR_TX: track 0.00 -> 16.4 mm, vias 0 -> 1
- net /RESET: track 60.0 -> 43.9 mm, vias 2 -> 1
- net N-0000036: track 0.00 -> 15.6 mm
