File: single-drive_pcb/single-drive_pcb.sch (KiCad schematic (older format))
At the start: 0 parts

Commit message: added most of the components to the schematic and did some basic wiring
Parts:
- added C?: 2.2uF, ~, symbol C
- added C?: 0.01uF, ~, symbol C
- added C?: 10uF, ~, symbol C
- added C? (x2): 22pF, ~, symbol C
- added C?: 1uF, ~, symbol C
- added IC?: DRV8834_SOP, symbol DRV8834_SOP
- added IC?: ATMEGA328P_TQFP, ~, symbol ATMEGA328P_TQFP
- added IC?: VCC_REG, ~, symbol VCC_REG
- added IC?: MAX3232, symbol MAX3232
- added J?: 8P8C_CUSTOM, ~, symbol 8P8C_CUSTOM
- added P?: AVR_ISP, ~, symbol AVR_ISP
- added R? (x4): 10k, ~, symbol R
- added S?: RST, ~, symbol SPST
- added Y?: 16MHz, ~, symbol CRYSTAL
Connections:
- net labels added: 232_RX, 232_TX, AVR_RX, AVR_TX, CONFIG, DIR, ENABLE, FAULT, GND, MISO, MOSI, MSEL0, MSEL1, RESET, SCK, SLEEP, STEP, VCC, VIN
- wire segments 0 -> 86
- no-connect marks 0 -> 6

Commit message: refactored schematic for wirelessly controlled battery powered application
Parts:
- removed IC?: VCC_REG, ~, symbol VCC_REG
- removed IC?: MAX3232, symbol MAX3232
- removed J?: 8P8C_CUSTOM, ~, symbol 8P8C_CUSTOM
- added C? (x3): 1uF, ~, symbol C
- added IC?: MIC5205, ~, symbol MIC5205
- added IC?: BLE112-A, ~, symbol BLE112-A
Connections:
- net labels added: VBAT
- net labels removed: 232_RX, 232_TX, VIN
- wire segments 86 -> 100
Other:
- moved on the sheet: C?, IC?, P?, R?, S?, Y?

Commit message: schematic coming along
Parts:
- added F?: 500mA, ~, symbol PTC
- added IC?: MCP4232, ~, symbol MCP42X2
- added R? (x4): 10kΩ, ~, symbol R
- added S?: BT_RST, ~, symbol SPST
- added VR? (x2): 10Ω, ~, symbol POT
- R? (x4): value 10k -> 10kΩ
Connections:
- net labels added: BT_DC, BT_DD, BT_RESET, R_SEL
- wire segments 100 -> 159
- no-connect marks 6 -> 13
Other:
- moved on the sheet: C?, IC?, R?

Commit message: schematic is done (until I find problems); moving on to footprint assignment
Parts:
- added BT1: LIPO, symbol LIPO
- added C10: 1uF, ~, symbol C
- added C11: 2.2uF, ~, symbol C
- added C12: 470pF, ~, symbol C
- added LED1: L1, ~, symbol LED
- added LED2: L2, ~, symbol LED
- added M1: STEPPER, ~, symbol 4PIN_HEADER
- added P2: CC_ISP, ~, symbol CC_ISP
- added R3, R4: 1kΩ, ~, symbol R
- R7: renamed from R?; value 10kΩ -> 22kΩ
- Y1: renamed from Y?; value 16MHz -> 8MHz
- gave numbers to parts that had none: 27
Connections:
- net BT_DC: now also P2.3 (DC)
- net BT_DD: now also P2.4 (DD)
- net BT_RESET: now also P2.7 (RST)
- net GND: now also C7.1, C8.1, C9.1, IC4.2 (GND), IC5.1 (GND), IC5.10 (GND), IC5.21 (GND), IC5.30 (GND), BT1.2 (-), C10.1, C11.2, C12.2, LED1.1 (C), LED2.1 (C), P2.1 (GND); no longer R6.2
- net VBAT: now also BT1.1 (+)
- net VCC: now also IC4.5 (VOUT), R6.2, C11.1, P2.2 (VCC), P2.9 (3.3V); no longer C5.2, IC3.20 (VINT)
- net at IC3.4 (AOUT1): now also M1.1
- net at IC3.6 (AOUT2): now also M1.2
- net at IC3.7 (BOUT2): now also M1.4
- net at IC3.9 (BOUT1): now also M1.3
- net at IC2.27 (PC4(ADC4/SDA/PCINT12)): now also R4.1
- net at IC2.28 (PC5(ADC5/SCL/PCINT13)): now also R3.1
- net at IC4.1 (VIN): now also F1.2, IC4.3 (EN), C10.2
- net at IC4.4 (BYP): now also C12.1
- new net: C5.2, IC3.20 (VINT)
- new net: LED1.2 (A), R3.2
- new net: LED2.2 (A), R4.2
- no-connect marks 13 -> 14
Other:
- note added: "MCU"
- note added: "Power"
- note added: "Stepper Driver"
- note added: "Wireless"
- moved on the sheet: C1, C2, C3, C4, C5, C6, C7, C8, C9, F1, IC1, IC2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

Commit message: hey, remember that time I completely forgot to add a charging circuit to my battery powered project?
Parts:
- added C13: 10uF, ~, symbol C
- added C14: 1uF, ~, symbol C
- added IC6: MAX1555, ~, symbol MAX1555
- added J1: MICROUSB, ~, symbol MICROUSB
- added LED3: PWR, ~, symbol LED
- added LED4: CHG, ~, symbol LED
- added R11, R12: 1kΩ, ~, symbol R
Connections:
- net GND: now also C13.1, C14.1, IC6.2 (GND), J1.5 (GND), LED3.1 (C)
- net VBAT: now also C14.2, IC6.5 (BAT), LED4.2 (A)
- net VCC: now also R11.2
- new net: LED3.2 (A), R11.1
- new net: C13.2, IC6.1 (VUSB), J1.1 (VBUS)
- new net: IC6.3 (~CHG~), R12.1
- new net: LED4.1 (C), R12.2
- no-connect marks 14 -> 17
Other:
- moved on the sheet: BT1, C10, C11, C12, C7, C8, C9, F1, IC4, IC5, P2, R10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

Commit message: schematic done and footprints assigned
Parts:
- added R13: 10kΩ, ~, symbol R
Connections:
- net GND: now also R13.1
- net at IC5.28 (P0_0), R10.2: no longer IC5.27 (P0_1)
- new net: IC5.27 (P0_1), R13.2
Other:
- moved on the sheet: BT1, C1, C10, C11, C12, C13, C14, C2, C3, C7, C8, C9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

Commit message: it's too late to be working on this
Connections:
- net AVR_RX: now also IC5.13 (P1_5(TX0_2)); no longer IC5.25 (P0_3(TX0_1))
- net AVR_TX: now also IC5.14 (P1_4(RX0_2)); no longer IC5.26 (P0_2(RX0_1))
- net at IC5.15 (P1_3), IC5.16 (P1_2), IC5.17 (P1_1)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: now also IC5.25 (P0_3(TX0_1)), IC5.26 (P0_2(RX0_1)); no longer IC5.13 (P1_5(TX0_2)), IC5.14 (P1_4(RX0_2))
Other:
- moved on the sheet: R9
Changed lines of the file:
@@
 Sheet 1 1
 Title "Single Stepper Driver Schematic"
-Date "19 jul 2013"
+Date "21 jul 2013"
 Rev "0.1"
 Comp "Copyright 2013 by Michael Cousins"
@@
 NoConn ~ 4400 2300
 NoConn ~ 4400 2200
-Text Label 9600 4950 2    60   ~ 0
+Text Label 9550 3850 2    60   ~ 0
 AVR_RX
-Text Label 9600 5050 2    60   ~ 0
-AVR_TX
 $Comp
 L R R10
@@
 L R R9
 U 1 1 51E99365
-P 9450 4200
-F 0 "R9" V 9500 4100 60  0000 C CNN
-F 1 "10kΩ" V 9400 4050 60  0000 C CNN
-F 2 "~" H 9450 4200 60  0000 C CNN
-F 3 "~" H 9450 4200 60  0000 C CNN
-	1    9450 4200
-	0    -1   -1   0
+P 9350 3400
+F 0 "R9" H 9450 3300 60  0000 C CNN
+F 1 "10kΩ" H 9200 3300 60  0000 C CNN
+F 2 "~" H 9350 3400 60  0000 C CNN
+F 3 "~" H 9350 3400 60  0000 C CNN
+	1    9350 3400
+	-1   0    0    1
 $EndComp
 $Comp
@@
 L GND #PWR022
 U 1 1 51E99DB4
-P 9450 3950
-F 0 "#PWR022" H 9450 3950 30  0001 C CNN
-F 1 "GND" H 9450 3880 30  0001 C CNN
-F 2 "" H 9450 3950 60  0000 C CNN
-F 3 "" H 9450 3950 60  0000 C CNN
-	1    9450 3950
-	-1   0    0    1
+P 9100 3400
+F 0 "#PWR022" H 9100 3400 30  0001 C CNN
+F 1 "GND" H 9100 3330 30  0001 C CNN
+F 2 "" H 9100 3400 60  0000 C CNN
+F 3 "" H 9100 3400 60  0000 C CNN
+	1    9100 3400
+	0    1    1    0
 $EndComp
 $Comp
@@
 	7400 5100 7750 5100
 Wire Wire Line
-	9600 5050 9150 5050
-Wire Wire Line
-	9600 4950 9150 4950
-Wire Wire Line
 	9250 5250 9150 5250
 Wire Wire Line
 	9250 4850 9150 4850
-Wire Wire Line
-	9250 3650 9250 4850
 Wire Wire Line
 	9250 4550 9150 4550
@@
 	9150 4350 9250 4350
 Wire Wire Line
-	9250 3650 9150 3650
+	9150 3650 9500 3650
 Wire Wire Line
 	9150 4250 9250 4250
@@
 Connection ~ 9250 4150
 Wire Wire Line
-	9150 4050 9250 4050
+	9150 4050 9650 4050
 Connection ~ 9250 4050
 Wire Wire Line
-	9150 3950 9250 3950
-Connection ~ 9250 3950
-Wire Wire Line
-	9150 3850 9250 3850
-Connection ~ 9250 3850
-Wire Wire Line
-	9150 3750 9250 3750
+	9150 3750 9650 3750
 Connection ~ 9250 3750
 Connection ~ 9250 4350
-Connection ~ 9250 4450
 Connection ~ 9250 4550
 Wire Wire Line
@@
 Wire Wire Line
 	7750 5300 7650 5300
-Connection ~ 9450 4450
-Wire Wire Line
-	9450 4450 9450 4350
-Wire Wire Line
-	9450 4050 9450 3950
 Wire Wire Line
 	4400 1950 4500 1950
@@
 $EndComp
 Wire Wire Line
-	9700 5700 9700 4450
-Wire Wire Line
-	7650 5700 9700 5700
-Wire Wire Line
-	9700 4450 9250 4450
-Wire Wire Line
 	9450 5550 9250 5550
 Wire Wire Line
 	9350 5550 9350 5450
 Connection ~ 9350 5550
+Text Label 9550 3950 2    60   ~ 0
+AVR_TX
+Wire Wire Line
+	9550 3850 9150 3850
+Wire Wire Line
+	9550 3950 9150 3950
+Wire Wire Line
+	9250 5050 9150 5050
+Wire Wire Line
+	9250 4050 9250 5050
+Wire Wire Line
+	9250 4950 9150 4950
+Connection ~ 9250 4950
+Connection ~ 9250 4850
+Wire Wire Line
+	9650 3750 9650 5700
+Wire Wire Line
+	9250 3750 9250 3650
+Wire Wire Line
+	9500 3650 9500 3400
+Connection ~ 9250 3650
+Wire Wire Line
+	9200 3400 9100 3400
+Connection ~ 9650 4050
+Wire Wire Line
+	9650 5700 7650 5700
 $EndSCHEMATC
